File: ECU-techPorsche88.kicad_pcb (KiCad board)
At the start: 4 copper layers, 160 x 118 mm, 0 parts

Commit message: up
Parts:
- added BT1: BATTERY_CR2032, Battery:BatteryHolder_Keystone_1060_1x2032, F.Cu at (133.3, 96.6)
- added C10: 10nF, Capacitor_SMD:C_0402_1005Metric, F.Cu at (167.8, 104.3)
- added C11: 10u, Capacitor_SMD:C_0603_1608Metric, F.Cu at (158.0, 64.9)
- added C12: 10u, Capacitor_SMD:C_0603_1608Metric, F.Cu at (162.0, 54.8)
- added C13: 10u, Capacitor_SMD:C_0603_1608Metric, F.Cu at (162.0, 57.3)
- added C14: 220nF, Capacitor_SMD:C_0402_1005Metric, F.Cu at (167.8, 106.3)
- added C15: 10u, Capacitor_SMD:C_0603_1608Metric, F.Cu at (162.0, 59.9)
- added C16: 100nF, Capacitor_SMD:C_0402_1005Metric, F.Cu at (170.7, 98.4)
- added C17: 100nF, Capacitor_SMD:C_0402_1005Metric, F.Cu at (170.7, 100.4)
- added C18: 10u, Capacitor_SMD:C_0603_1608Metric, F.Cu at (162.0, 62.4)
- added C19: 100nF, Capacitor_SMD:C_0402_1005Metric, F.Cu at (170.7, 102.4)
- added C20: 10u, Capacitor_SMD:C_0603_1608Metric, F.Cu at (162.0, 64.9)
- added C21: 100nF, Capacitor_SMD:C_0402_1005Metric, F.Cu at (170.7, 104.3)
- added C23: 100nF, Capacitor_SMD:C_0402_1005Metric, F.Cu at (170.7, 106.3)
- added C3: 100nF, Capacitor_SMD:C_0402_1005Metric, F.Cu at (167.8, 98.4)
- added C4: 10u, Capacitor_SMD:C_0603_1608Metric, F.Cu at (158.0, 54.8)
- added C5: 10u, Capacitor_SMD:C_0603_1608Metric, F.Cu at (158.0, 57.3)
- added C6: 10u, Capacitor_SMD:C_0603_1608Metric, F.Cu at (158.0, 59.9)
- added C7: 100nF, Capacitor_SMD:C_0402_1005Metric, F.Cu at (167.8, 100.4)
- added C8: 5.6nF, Capacitor_SMD:C_0402_1005Metric, F.Cu at (167.8, 102.4)
- added C9: 10u, Capacitor_SMD:C_0603_1608Metric, F.Cu at (158.0, 62.4)
- added D1: B5819W, Diode_SMD:D_SOD-123, F.Cu at (135.4, 109.5)
- added D10: LED-RED-0603, LED_SMD:LED_0603_1608Metric, F.Cu at (118.3, 111.7)
- added D11: 1N4148WS, Diode_SMD:D_SOD-323, F.Cu at (145.3, 62.1)
- added D12: LED-RED-0603, LED_SMD:LED_0603_1608Metric, F.Cu at (118.3, 114.3)
- added D13: 1N4148WS, Diode_SMD:D_SOD-323, F.Cu at (145.3, 65.0)
- added D14: LED-RED-0603, LED_SMD:LED_0603_1608Metric, F.Cu at (118.3, 116.9)
- added D15: 1N4148WS, Diode_SMD:D_SOD-323, F.Cu at (149.6, 50.3)
- added D16: LED-RED-0603, LED_SMD:LED_0603_1608Metric, F.Cu at (118.3, 119.5)
- added D17: 1N4148WS, Diode_SMD:D_SOD-323, F.Cu at (149.6, 53.2)
- added D18: LED-RED-0603, LED_SMD:LED_0603_1608Metric, F.Cu at (118.3, 122.1)
- added D19: 1N4148WS, Diode_SMD:D_SOD-323, F.Cu at (149.6, 56.2)
- added D2: B5819W, Diode_SMD:D_SOD-123, F.Cu at (135.4, 112.9)
- added D20: LED-RED-0603, LED_SMD:LED_0603_1608Metric, F.Cu at (122.4, 109.1)
- added D21: 1N4148WS, Diode_SMD:D_SOD-323, F.Cu at (149.6, 59.1)
- added D22: LED-RED-0603, LED_SMD:LED_0603_1608Metric, F.Cu at (122.4, 111.7)
- added D23: LED-BLUE-0603, LED_SMD:LED_0603_1608Metric, F.Cu at (122.4, 114.3)
- added D24: LED-BLUE-0603, LED_SMD:LED_0603_1608Metric, F.Cu at (122.4, 116.9)
- added D25: LED-BLUE-0603, LED_SMD:LED_0603_1608Metric, F.Cu at (122.4, 119.5)
- added D26: LED-BLUE-0603, LED_SMD:LED_0603_1608Metric, F.Cu at (122.4, 122.1)
- added D27: LED-BLUE-0603, LED_SMD:LED_0603_1608Metric, F.Cu at (126.4, 109.1)
- added D28: LED-BLUE-0603, LED_SMD:LED_0603_1608Metric, F.Cu at (126.4, 111.7)
- added D29: LED-BLUE-0603, LED_SMD:LED_0603_1608Metric, F.Cu at (126.4, 114.3)
- added D3: 1N4148WS, Diode_SMD:D_SOD-323, F.Cu at (145.3, 50.3)
- added D30: LED-BLUE-0603, LED_SMD:LED_0603_1608Metric, F.Cu at (126.4, 116.9)
- added D31: LED-GREEN-0603, LED_SMD:LED_0603_1608Metric, F.Cu at (126.4, 119.5)
- added D32: LED-GREEN-0603, LED_SMD:LED_0603_1608Metric, F.Cu at (126.4, 122.1)
- added D33: LED-GREEN-0603, LED_SMD:LED_0603_1608Metric, F.Cu at (130.5, 109.1)
- added D34: 1N4148WS, Diode_SMD:D_SOD-323, F.Cu at (149.6, 62.1)
- added D35: LED-GREEN-0603, LED_SMD:LED_0603_1608Metric, F.Cu at (130.5, 111.7)
- added D36: 1N4148WS, Diode_SMD:D_SOD-323, F.Cu at (149.6, 65.0)
- added D37: LED-RED-0603, LED_SMD:LED_0603_1608Metric, F.Cu at (130.5, 114.3)
- added D38: 1N4148WS, Diode_SMD:D_SOD-323, F.Cu at (153.9, 50.3)
- added D39: LED-RED-0603, LED_SMD:LED_0603_1608Metric, F.Cu at (130.5, 116.9)
- added D4: 1N4148WS, Diode_SMD:D_SOD-323, F.Cu at (145.3, 53.2)
- added D40: 1N4148WS, Diode_SMD:D_SOD-323, F.Cu at (153.9, 53.2)
- added D41: LED-WHITE-0603, LED_SMD:LED_0603_1608Metric, F.Cu at (130.5, 119.5)
- added D42: 1N4148WS, Diode_SMD:D_SOD-323, F.Cu at (153.9, 56.2)
- added D5: B5819W, Diode_SMD:D_SOD-123, F.Cu at (135.4, 116.2)
- added D6: B5819W, Diode_SMD:D_SOD-123, F.Cu at (135.4, 119.6)
- added D7: 1N4148WS, Diode_SMD:D_SOD-323, F.Cu at (145.3, 56.2)
- added D8: LED-RED-0603, LED_SMD:LED_0603_1608Metric, F.Cu at (118.3, 109.1)
- added D9: 1N4148WS, Diode_SMD:D_SOD-323, F.Cu at (145.3, 59.1)
- added H1: MountingHole, MountingHole:MountingHole_4.3mm_M4_DIN965, F.Cu at (147.6, 71.0)
- added H2: MountingHole, MountingHole:MountingHole_4.3mm_M4_DIN965, F.Cu at (147.6, 80.1)
- added J1: Conn_01x05, Connector_PinHeader_2.54mm:PinHeader_1x05_P2.54mm_Vertical, F.Cu at (169.0, 68.8)
- added J10: Conn_01x05, Connector_PinHeader_2.00mm:PinHeader_1x05_P2.00mm_Vertical, F.Cu at (168.4, 87.4)
- added J2: MiniFit, Connector_Molex:Molex_Mini-Fit_Jr_5569-02A2_2x01_P4.20mm_Horizontal, F.Cu at (162.7, 100.3)
- added J3: VRIN1, Connector_PinHeader_1.00mm:PinHeader_1x01_P1.00mm_Vertical, F.Cu at (118.0, 50.3)
- added J4: VRIN2, Connector_PinHeader_1.00mm:PinHeader_1x01_P1.00mm_Vertical, F.Cu at (118.0, 53.4)
- added J6: VROUT1, Connector_PinHeader_1.00mm:PinHeader_1x01_P1.00mm_Vertical, F.Cu at (118.0, 56.4)
- added J7: ETB, Connector_PinHeader_2.54mm:PinHeader_1x06_P2.54mm_Vertical, F.Cu at (164.3, 68.8)
- added J8: PPS, Connector_PinHeader_2.54mm:PinHeader_1x04_P2.54mm_Vertical, F.Cu at (166.3, 55.9)
- added KNOCK_RAW1: IN_KNOCK1_RAW, Connector_PinHeader_1.00mm:PinHeader_1x01_P1.00mm_Vertical, F.Cu at (118.0, 59.5)
- added KNOCK_RAW2: IN_KNOCK2_RAW, Connector_PinHeader_1.00mm:PinHeader_1x01_P1.00mm_Vertical, F.Cu at (118.0, 62.5)
- added MMCU1: MMCU, Connector_PinHeader_1.00mm:PinHeader_1x01_P1.00mm_Vertical, F.Cu at (118.0, 65.6)
- added MMCU10: MMCU, Connector_PinHeader_1.00mm:PinHeader_1x01_P1.00mm_Vertical, F.Cu at (121.3, 56.4)
- added MMCU11: MMCU, Connector_PinHeader_1.00mm:PinHeader_1x01_P1.00mm_Vertical, F.Cu at (121.3, 59.5)
- added MMCU12: MMCU, Connector_PinHeader_1.00mm:PinHeader_1x01_P1.00mm_Vertical, F.Cu at (121.3, 62.5)
- added MMCU13: MMCU, Connector_PinHeader_1.00mm:PinHeader_1x01_P1.00mm_Vertical, F.Cu at (121.3, 65.6)
- added MMCU14: MMCU, Connector_PinHeader_1.00mm:PinHeader_1x01_P1.00mm_Vertical, F.Cu at (121.3, 68.6)
- added MMCU15: MMCU, Connector_PinHeader_1.00mm:PinHeader_1x01_P1.00mm_Vertical, F.Cu at (121.3, 71.7)
- added MMCU16: MMCU, Connector_PinHeader_1.00mm:PinHeader_1x01_P1.00mm_Vertical, F.Cu at (121.3, 74.7)
- added MMCU17: MMCU, Connector_PinHeader_1.00mm:PinHeader_1x01_P1.00mm_Vertical, F.Cu at (121.3, 77.8)
- added MMCU18: MMCU, Connector_PinHeader_1.00mm:PinHeader_1x01_P1.00mm_Vertical, F.Cu at (121.3, 80.8)
- added MMCU19: MMCU, Connector_PinHeader_1.00mm:PinHeader_1x01_P1.00mm_Vertical, F.Cu at (121.3, 83.9)
- added MMCU2: MMCU, Connector_PinHeader_1.00mm:PinHeader_1x01_P1.00mm_Vertical, F.Cu at (118.0, 68.6)
- added MMCU20: MMCU, Connector_PinHeader_1.00mm:PinHeader_1x01_P1.00mm_Vertical, F.Cu at (124.7, 50.3)
- added MMCU21: MMCU, Connector_PinHeader_1.00mm:PinHeader_1x01_P1.00mm_Vertical, F.Cu at (124.7, 53.4)
- added MMCU22: MMCU, Connector_PinHeader_1.00mm:PinHeader_1x01_P1.00mm_Vertical, F.Cu at (124.7, 56.4)
- added MMCU23: MMCU, Connector_PinHeader_1.00mm:PinHeader_1x01_P1.00mm_Vertical, F.Cu at (124.7, 59.5)
- added MMCU24: MMCU, Connector_PinHeader_1.00mm:PinHeader_1x01_P1.00mm_Vertical, F.Cu at (124.7, 62.5)
- added MMCU25: MMCU, Connector_PinHeader_1.00mm:PinHeader_1x01_P1.00mm_Vertical, F.Cu at (124.7, 65.6)
- added MMCU26: MMCU, Connector_PinHeader_1.00mm:PinHeader_1x01_P1.00mm_Vertical, F.Cu at (124.7, 68.6)
- added MMCU27: MMCU, Connector_PinHeader_1.00mm:PinHeader_1x01_P1.00mm_Vertical, F.Cu at (124.7, 71.7)
- added MMCU28: MMCU, Connector_PinHeader_1.00mm:PinHeader_1x01_P1.00mm_Vertical, F.Cu at (124.7, 74.7)
- added MMCU29: MMCU, Connector_PinHeader_1.00mm:PinHeader_1x01_P1.00mm_Vertical, F.Cu at (124.7, 77.8)
- added MMCU3: MMCU, Connector_PinHeader_1.00mm:PinHeader_1x01_P1.00mm_Vertical, F.Cu at (118.0, 71.7)
- added MMCU30: MMCU, Connector_PinHeader_1.00mm:PinHeader_1x01_P1.00mm_Vertical, F.Cu at (124.7, 80.8)
- added MMCU31: MMCU, Connector_PinHeader_1.00mm:PinHeader_1x01_P1.00mm_Vertical, F.Cu at (124.7, 83.9)
- added MMCU4: MMCU, Connector_PinHeader_1.00mm:PinHeader_1x01_P1.00mm_Vertical, F.Cu at (118.0, 74.7)
- added MMCU5: MMCU, Connector_PinHeader_1.00mm:PinHeader_1x01_P1.00mm_Vertical, F.Cu at (118.0, 77.8)
- added MMCU6: MMCU, Connector_PinHeader_1.00mm:PinHeader_1x01_P1.00mm_Vertical, F.Cu at (118.0, 80.8)
- added MMCU7: MMCU, Connector_PinHeader_1.00mm:PinHeader_1x01_P1.00mm_Vertical, F.Cu at (118.0, 83.9)
- added MMCU8: MMCU, Connector_PinHeader_1.00mm:PinHeader_1x01_P1.00mm_Vertical, F.Cu at (121.3, 50.3)
- added MMCU9: MMCU, Connector_PinHeader_1.00mm:PinHeader_1x01_P1.00mm_Vertical, F.Cu at (121.3, 53.4)
- added P1: P, Connector_Pin:Pin_D1.0mm_L10.0mm, F.Cu at (161.0, 110.7)
- added P2: P, Connector_Pin:Pin_D1.0mm_L10.0mm, F.Cu at (161.0, 114.8)
- added P3: P, Connector_Pin:Pin_D1.0mm_L10.0mm, F.Cu at (165.0, 110.7)
- added P4: P, Connector_Pin:Pin_D1.0mm_L10.0mm, F.Cu at (165.0, 114.8)
- added P5: P, Connector_Pin:Pin_D1.0mm_L10.0mm, F.Cu at (169.1, 110.7)
- added P6: P, Connector_Pin:Pin_D1.0mm_L10.0mm, F.Cu at (169.1, 114.8)
- added Q1: NGD8201AN, Package_TO_SOT_SMD:TO-252-2, F.Cu at (111.1, 52.8)
- added Q10: AUIPS2041LTR, Package_TO_SOT_SMD:SOT-223, F.Cu at (157.1, 79.0)
- added Q2: NGD8201AN, Package_TO_SOT_SMD:TO-252-2, F.Cu at (111.1, 60.9)
- added Q3: NGD8201AN, Package_TO_SOT_SMD:TO-252-2, F.Cu at (111.1, 68.9)
- added Q4: NGD8201AN, Package_TO_SOT_SMD:TO-252-2, F.Cu at (111.1, 77.0)
- added Q5: NGD8201AN, Package_TO_SOT_SMD:TO-252-2, F.Cu at (111.1, 85.0)
- added Q6: NGD8201AN, Package_TO_SOT_SMD:TO-252-2, F.Cu at (111.1, 93.1)
- added Q7: NGD8201AN, Package_TO_SOT_SMD:TO-252-2, F.Cu at (111.1, 101.1)
- added Q8: NGD8201AN, Package_TO_SOT_SMD:TO-252-2, F.Cu at (111.1, 109.2)
- added Q9: AUIPS2041LTR, Package_TO_SOT_SMD:SOT-223, F.Cu at (157.1, 70.7)
- added R1: DNP, Resistor_SMD:R_2512_6332Metric, F.Cu at (154.6, 87.8)
- added R12: DNP, Resistor_SMD:R_2512_6332Metric, F.Cu at (154.6, 112.3)
- added R13: DNP, Resistor_SMD:R_0402_1005Metric, F.Cu at (139.7, 108.8)
- added R14: DNP, Resistor_SMD:R_0402_1005Metric, F.Cu at (139.7, 110.8)
- added R15: 100k, Resistor_SMD:R_0402_1005Metric, F.Cu at (139.7, 112.8)
- added R16: 100, Resistor_SMD:R_0402_1005Metric, F.Cu at (139.7, 114.8)
- added R17: 10k, Resistor_SMD:R_0402_1005Metric, F.Cu at (139.7, 116.8)
- added R18: DNP, Resistor_SMD:R_2512_6332Metric, F.Cu at (154.6, 117.2)
- added R21: DNP, Resistor_SMD:R_2512_6332Metric, F.Cu at (154.6, 122.1)
- added R24: 10k, Resistor_SMD:R_0402_1005Metric, F.Cu at (142.7, 108.8)
- added R25: 10k, Resistor_SMD:R_0402_1005Metric, F.Cu at (142.7, 110.8)
- added R31: 1k6, Resistor_SMD:R_0402_1005Metric, F.Cu at (142.7, 112.8)
- added R32: 750R, Resistor_SMD:R_0402_1005Metric, F.Cu at (142.7, 114.8)
- added R33: 5k1, Resistor_SMD:R_0402_1005Metric, F.Cu at (142.7, 116.8)
- added R34: 5k1, Resistor_SMD:R_0402_1005Metric, F.Cu at (145.6, 108.8)
- added R35: 5k1, Resistor_SMD:R_0402_1005Metric, F.Cu at (145.6, 110.8)
- added R36: 20k, Resistor_SMD:R_0402_1005Metric, F.Cu at (145.6, 112.8)
- added R37: 4.7k, Resistor_SMD:R_0402_1005Metric, F.Cu at (145.6, 114.8)
- added R4: DNP, Resistor_SMD:R_2512_6332Metric, F.Cu at (154.6, 92.7)
- added R5: DNP, Resistor_SMD:R_2512_6332Metric, F.Cu at (154.6, 97.6)
- added R8: DNP, Resistor_SMD:R_2512_6332Metric, F.Cu at (154.6, 102.5)
- added R9: DNP, Resistor_SMD:R_2512_6332Metric, F.Cu at (154.6, 107.4)
- added RN1: 4.7k, Resistor_SMD:R_Array_Concave_4x0603, F.Cu at (158.1, 51.2)
- added RN2: 4.7k, Resistor_SMD:R_Array_Concave_4x0603, F.Cu at (162.2, 51.2)
- added RN3: 1k, Resistor_SMD:R_Array_Concave_4x0603, F.Cu at (166.3, 51.2)
- added RN4: 1k, Resistor_SMD:R_Array_Concave_4x0603, F.Cu at (170.5, 51.2)
- added TP1: TestPoint, TestPoint:TestPoint_Pad_D1.0mm, F.Cu at (170.2, 55.1)
- added TP2: TestPoint, TestPoint:TestPoint_Pad_D1.0mm, F.Cu at (170.2, 58.2)
- added TP3: TestPoint, TestPoint:TestPoint_Pad_D1.0mm, F.Cu at (170.2, 61.2)
- added TP4: TestPoint, TestPoint:TestPoint_Pad_D1.0mm, F.Cu at (170.2, 64.3)
- added U2: TLS115_SON, Package_SON:HVSON-8-1EP_3x3mm_P0.65mm_EP1.6x2.4mm, F.Cu at (107.2, 115.5)
- added U3: MCP6002-xSN, Package_SO:SOIC-8_3.9x4.9mm_P1.27mm, F.Cu at (142.5, 121.1)
- added U6: MPXA6115A, Package_SO:SSO-8_6.8x5.9mm_P1.27mm_Clearance7mm, F.Cu at (165.1, 120.5)
- added U8: LPS25HB, Package_LGA:ST_HLGA-10_2.5x2.5mm_P0.6mm_LayoutBorder3x2y, F.Cu at (112.0, 115.5)
- added VIN1: VIN9, Connector_PinHeader_1.00mm:PinHeader_1x01_P1.00mm_Vertical, F.Cu at (128.0, 50.3)
- added VIN10: VIN16, Connector_PinHeader_1.00mm:PinHeader_1x01_P1.00mm_Vertical, F.Cu at (128.0, 77.8)
- added VIN11: VIN17, Connector_PinHeader_1.00mm:PinHeader_1x01_P1.00mm_Vertical, F.Cu at (128.0, 80.8)
- added VIN2: VIN8, Connector_PinHeader_1.00mm:PinHeader_1x01_P1.00mm_Vertical, F.Cu at (128.0, 53.4)
- added VIN3: VIN8, Connector_PinHeader_1.00mm:PinHeader_1x01_P1.00mm_Vertical, F.Cu at (128.0, 56.4)
- added VIN4: VIN8, Connector_PinHeader_1.00mm:PinHeader_1x01_P1.00mm_Vertical, F.Cu at (128.0, 59.5)
- added VIN5: VIN8, Connector_PinHeader_1.00mm:PinHeader_1x01_P1.00mm_Vertical, F.Cu at (128.0, 62.5)
- added VIN6: VIN8, Connector_PinHeader_1.00mm:PinHeader_1x01_P1.00mm_Vertical, F.Cu at (128.0, 65.6)
- added VIN7: VIN8, Connector_PinHeader_1.00mm:PinHeader_1x01_P1.00mm_Vertical, F.Cu at (128.0, 68.6)
- added VIN8: VIN8, Connector_PinHeader_1.00mm:PinHeader_1x01_P1.00mm_Vertical, F.Cu at (128.0, 71.7)
- added VIN9: VIN10, Connector_PinHeader_1.00mm:PinHeader_1x01_P1.00mm_Vertical, F.Cu at (128.0, 74.7)
- added VOUT1: VOUT4, Connector_PinHeader_1.00mm:PinHeader_1x01_P1.00mm_Vertical, F.Cu at (128.0, 83.9)
- added VOUT10: VOUT4, Connector_PinHeader_1.00mm:PinHeader_1x01_P1.00mm_Vertical, F.Cu at (131.4, 74.7)
- added VOUT11: VOUT4, Connector_PinHeader_1.00mm:PinHeader_1x01_P1.00mm_Vertical, F.Cu at (131.4, 77.8)
- added VOUT12: VOUT4, Connector_PinHeader_1.00mm:PinHeader_1x01_P1.00mm_Vertical, F.Cu at (131.4, 80.8)
- added VOUT13: VOUT5, Connector_PinHeader_1.00mm:PinHeader_1x01_P1.00mm_Vertical, F.Cu at (131.4, 83.9)
- added VOUT14: VOUT4, Connector_PinHeader_1.00mm:PinHeader_1x01_P1.00mm_Vertical, F.Cu at (134.7, 50.3)
- added VOUT15: VOUT4, Connector_PinHeader_1.00mm:PinHeader_1x01_P1.00mm_Vertical, F.Cu at (134.7, 53.4)
- added VOUT16: VOUT4, Connector_PinHeader_1.00mm:PinHeader_1x01_P1.00mm_Vertical, F.Cu at (134.7, 56.4)
- added VOUT17: VOUT4, Connector_PinHeader_1.00mm:PinHeader_1x01_P1.00mm_Vertical, F.Cu at (134.7, 59.5)
- added VOUT18: VOUT6, Connector_PinHeader_1.00mm:PinHeader_1x01_P1.00mm_Vertical, F.Cu at (134.7, 62.5)
- added VOUT19: VOUT4, Connector_PinHeader_1.00mm:PinHeader_1x01_P1.00mm_Vertical, F.Cu at (134.7, 65.6)
- added VOUT2: VOUT4, Connector_PinHeader_1.00mm:PinHeader_1x01_P1.00mm_Vertical, F.Cu at (131.4, 50.3)
- added VOUT20: VOUT4, Connector_PinHeader_1.00mm:PinHeader_1x01_P1.00mm_Vertical, F.Cu at (134.7, 68.6)
- added VOUT21: VOUT4, Connector_PinHeader_1.00mm:PinHeader_1x01_P1.00mm_Vertical, F.Cu at (134.7, 71.7)
- added VOUT22: VOUT4, Connector_PinHeader_1.00mm:PinHeader_1x01_P1.00mm_Vertical, F.Cu at (134.7, 74.7)
- added VOUT23: VOUT4, Connector_PinHeader_1.00mm:PinHeader_1x01_P1.00mm_Vertical, F.Cu at (134.7, 77.8)
- added VOUT24: VOUT4, Connector_PinHeader_1.00mm:PinHeader_1x01_P1.00mm_Vertical, F.Cu at (134.7, 80.8)
- added VOUT25: VOUT4, Connector_PinHeader_1.00mm:PinHeader_1x01_P1.00mm_Vertical, F.Cu at (134.7, 83.9)
- added VOUT26: VOUT4, Connector_PinHeader_1.00mm:PinHeader_1x01_P1.00mm_Vertical, F.Cu at (138.1, 50.3)
- added VOUT3: VOUT4, Connector_PinHeader_1.00mm:PinHeader_1x01_P1.00mm_Vertical, F.Cu at (131.4, 53.4)
- added VOUT4: VOUT4, Connector_PinHeader_1.00mm:PinHeader_1x01_P1.00mm_Vertical, F.Cu at (131.4, 56.4)
- added VOUT5: VOUT4, Connector_PinHeader_1.00mm:PinHeader_1x01_P1.00mm_Vertical, F.Cu at (131.4, 59.5)
- added VOUT6: VOUT4, Connector_PinHeader_1.00mm:PinHeader_1x01_P1.00mm_Vertical, F.Cu at (131.4, 62.5)
- added VOUT7: VOUT4, Connector_PinHeader_1.00mm:PinHeader_1x01_P1.00mm_Vertical, F.Cu at (131.4, 65.6)
- added VOUT8: VOUT4, Connector_PinHeader_1.00mm:PinHeader_1x01_P1.00mm_Vertical, F.Cu at (131.4, 68.6)
- added VOUT9: VOUT4, Connector_PinHeader_1.00mm:PinHeader_1x01_P1.00mm_Vertical, F.Cu at (131.4, 71.7)
- added cr1: cr, Connector_PinHeader_1.00mm:PinHeader_1x01_P1.00mm_Vertical, F.Cu at (138.1, 53.4)
- added cr10: cr, Connector_PinHeader_1.00mm:PinHeader_1x01_P1.00mm_Vertical, F.Cu at (138.1, 80.8)
- added cr11: cr, Connector_PinHeader_1.00mm:PinHeader_1x01_P1.00mm_Vertical, F.Cu at (138.1, 83.9)
- added cr12: cr, Connector_PinHeader_1.00mm:PinHeader_1x01_P1.00mm_Vertical, F.Cu at (141.4, 50.3)
- added cr13: cr, Connector_PinHeader_1.00mm:PinHeader_1x01_P1.00mm_Vertical, F.Cu at (141.4, 53.4)
- added cr14: cr, Connector_PinHeader_1.00mm:PinHeader_1x01_P1.00mm_Vertical, F.Cu at (141.4, 56.4)
- added cr15: cr, Connector_PinHeader_1.00mm:PinHeader_1x01_P1.00mm_Vertical, F.Cu at (141.4, 59.5)
- added cr16: cr, Connector_PinHeader_1.00mm:PinHeader_1x01_P1.00mm_Vertical, F.Cu at (141.4, 62.5)
- added cr17: cr, Connector_PinHeader_1.00mm:PinHeader_1x01_P1.00mm_Vertical, F.Cu at (141.4, 65.6)
- added cr18: cr, Connector_PinHeader_1.00mm:PinHeader_1x01_P1.00mm_Vertical, F.Cu at (141.4, 68.6)
- added cr19: cr, Connector_PinHeader_1.00mm:PinHeader_1x01_P1.00mm_Vertical, F.Cu at (141.4, 71.7)
- added cr2: cr, Connector_PinHeader_1.00mm:PinHeader_1x01_P1.00mm_Vertical, F.Cu at (138.1, 56.4)
- added cr20: cr, Connector_PinHeader_1.00mm:PinHeader_1x01_P1.00mm_Vertical, F.Cu at (141.4, 74.7)
- added cr21: cr, Connector_PinHeader_1.00mm:PinHeader_1x01_P1.00mm_Vertical, F.Cu at (141.4, 77.8)
- added cr22: cr, Connector_PinHeader_1.00mm:PinHeader_1x01_P1.00mm_Vertical, F.Cu at (141.4, 80.8)
- added cr3: cr, Connector_PinHeader_1.00mm:PinHeader_1x01_P1.00mm_Vertical, F.Cu at (138.1, 59.5)
- added cr4: cr, Connector_PinHeader_1.00mm:PinHeader_1x01_P1.00mm_Vertical, F.Cu at (138.1, 62.5)
- added cr5: cr, Connector_PinHeader_1.00mm:PinHeader_1x01_P1.00mm_Vertical, F.Cu at (138.1, 65.6)
- added cr6: cr, Connector_PinHeader_1.00mm:PinHeader_1x01_P1.00mm_Vertical, F.Cu at (138.1, 68.6)
- added cr7: cr, Connector_PinHeader_1.00mm:PinHeader_1x01_P1.00mm_Vertical, F.Cu at (138.1, 71.7)
- added cr8: cr, Connector_PinHeader_1.00mm:PinHeader_1x01_P1.00mm_Vertical, F.Cu at (138.1, 74.7)
- added cr9: cr, Connector_PinHeader_1.00mm:PinHeader_1x01_P1.00mm_Vertical, F.Cu at (138.1, 77.8)
