File: ECU-techPorsche88.kicad_sch (KiCad schematic)
At the start: 304 parts, among them J1 Conn_01x05, J10 Conn_01x05, J11 USB_B_Mini, J2 MiniFit, J3 VRIN1, J4 VRIN2, J5 AudioJack_THR, J6 VROUT1, J7 ETB, J8 PPS, J9 XH-8A, M1 Module-power12-0.2, M10 Module-sd-0.1, M11 Module-can-0.1, M12 Module-wbo-0.3, M13 Module-can-0.1, M2 Module-power5-0.2, M3 Module-knock-0.1, M4 Module-knock-0.1, M5 Module-vr-0.1, M6 Module-output-0.3, M7 Module-input-0.1, M8 Module-ign8-0.2, M9 Module-mcu144-0.6, P1 P, P2 P, P3 P, P4 P, P5 P, P6 P, Q1 NGD8201AN, Q10 AUIPS2041LTR, Q2 NGD8201AN, Q3 NGD8201AN, Q4 NGD8201AN, Q5 NGD8201AN, Q6 NGD8201AN, Q7 NGD8201AN, Q8 NGD8201AN, Q9 AUIPS2041LTR, SW1 Button_SPST, SW2 Button_SPST, U1 TLS115_SOIC, U2 TLS115_SON, U3 MCP6002-xSN, U4 L6205PD, U5 MPX4_MAP, U6 MPXA6115A, U7 LIS2DW12TR, U8 LPS25HB

Commit message: up
Parts:
- M1: symbol hellen-one-power12-0.2:Module-power12-0.2 -> power12-0.2:Module-power12-0.2
- M10: symbol hellen-one-sd-0.1:Module-sd-0.1 -> sd-0.1:Module-sd-0.1
- M11, M13: symbol hellen-one-can-0.1:Module-can-0.1 -> can-0.1:Module-can-0.1
- M12: symbol hellen-one-wbo-0.3:Module-wbo-0.3 -> wbo-0.3:Module-wbo-0.3
- M2: symbol hellen-one-power5-0.2:Module-power5-0.2 -> power5-0.2:Module-power5-0.2
- M3, M4: symbol hellen-one-knock-0.1:Module-knock-0.1 -> knock-0.1:Module-knock-0.1
- M6: symbol hellen-one-output-0.3:Module-output-0.3 -> output-0.3:Module-output-0.3
- M7: symbol hellen-one-input-0.1:Module-input-0.1 -> input-0.1:Module-input-0.1
- M8: symbol hellen-one-ign8-0.2:Module-ign8-0.2 -> ign8-0.2:Module-ign8-0.2
- M9: symbol hellen-one-mcu-0.6:Module-mcu-0.6 -> mcu-0.6:Module-mcu-0.6
- U5: footprint rusefi_lib:MPX-4_MAP -> hellen-one-common:MPXH6400A-SSOP8; symbol MPX-4_MAP:MPX4_MAP -> hellen-one-common:MPX4_MAP; LCSC (none) -> C511770
Connections:
- net +5VA: now also U5.2 (Vs); no longer U5.3 (VCC)
- net GND: now also U5.3 (GND); no longer U5.2 (GND)
- net IN_MAP2: now also U5.4 (Vout); no longer U5.1 (VOUT)
- no-connect marks 41 -> 43
Other:
- title: Porsche88 -> (none)
- moved on the sheet: C7

Commit message: neu
Parts:
- renumbered C7 to C4, C4 to C5, C5 to C6, C6 to C7
Changed lines of the file:
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@@
 		(on_board yes)
 		(dnp no)
-		(property "Reference" "C5"
+		(property "Reference" "C6"
 			(at 332.232 338.582 90)
 			(effects
@@
 			(project "ECU-techPorsche88"
 				(path "/2a08f213-b835-4bb3-95c3-61aa4df68063"
-					(reference "C5")
+					(reference "C6")
 					(unit 1)
 				)
@@
 		(on_board yes)
 		(dnp no)
-		(property "Reference" "C4"
+		(property "Reference" "C5"
 			(at 332.232 322.072 90)
 			(effects
@@
 			(project "ECU-techPorsche88"
 				(path "/2a08f213-b835-4bb3-95c3-61aa4df68063"
-					(reference "C4")
+					(reference "C5")
 					(unit 1)
 				)
@@
 		(on_board yes)
 		(dnp no)
-		(property "Reference" "C6"
+		(property "Reference" "C7"
 			(at 338.582 410.972 90)
 			(effects
@@
 			(project "ECU-techPorsche88"
 				(path "/2a08f213-b835-4bb3-95c3-61aa4df68063"
-					(reference "C6")
+					(reference "C7")
 					(unit 1)
 				)
@@
 		(dnp no)
 		(fields_autoplaced yes)
-		(property "Reference" "#PWR043"
+		(property "Reference" "#PWR037"
 			(at 327.406 275.336 0)
 			(effects
@@
 			(project "ECU-techPorsche88"
 				(path "/2a08f213-b835-4bb3-95c3-61aa4df68063"
-					(reference "#PWR043")
+					(reference "#PWR037")
 					(unit 1)
 				)
@@
 		(on_board yes)
 		(dnp no)
-		(property "Reference" "C7"
+		(property "Reference" "C4"
 			(at 323.215 277.9776 0)
 			(effects
@@
 			(project "ECU-techPorsche88"
 				(path "/2a08f213-b835-4bb3-95c3-61aa4df68063"
-					(reference "C7")
+					(reference "C4")
 					(unit 1)
 				)
@@
 		(on_board yes)
 		(dnp no)
-		(property "Reference" "#PWR039"
+		(property "Reference" "#PWR042"
 			(at 345.694 266.192 0)
 			(effects
@@
 			(project "ECU-techPorsche88"
 				(path "/2a08f213-b835-4bb3-95c3-61aa4df68063"
-					(reference "#PWR039")
+					(reference "#PWR042")
 					(unit 1)
 				)
@@
 		(on_board yes)
 		(dnp no)
-		(property "Reference" "#PWR041"
+		(property "Reference" "#PWR039"
 			(at 326.136 289.306 0)
 			(effects
@@
 			(project "ECU-techPorsche88"
 				(path "/2a08f213-b835-4bb3-95c3-61aa4df68063"
-					(reference "#PWR041")
+					(reference "#PWR039")
 					(unit 1)
 				)
@@
 		(on_board yes)
 		(dnp no)
-		(property "Reference" "#PWR040"
+		(property "Reference" "#PWR041"
 			(at 343.662 341.122 0)
 			(effects
@@
 			(project "ECU-techPorsche88"
 				(path "/2a08f213-b835-4bb3-95c3-61aa4df68063"
-					(reference "#PWR040")
+					(reference "#PWR041")
 					(unit 1)
 				)
@@
 		(on_board yes)
 		(dnp no)
-		(property "Reference" "#PWR038"
+		(property "Reference" "#PWR040"
 			(at 342.392 399.542 0)
 			(effects
@@
 			(project "ECU-techPorsche88"
 				(path "/2a08f213-b835-4bb3-95c3-61aa4df68063"
-					(reference "#PWR038")
+					(reference "#PWR040")
 					(unit 1)
 				)
@@
 		(on_board yes)
 		(dnp no)
-		(property "Reference" "#PWR037"
+		(property "Reference" "#PWR038"
 			(at 325.882 64.262 0)
 			(effects
@@
 			(project "ECU-techPorsche88"
 				(path "/2a08f213-b835-4bb3-95c3-61aa4df68063"
-					(reference "#PWR037")
+					(reference "#PWR038")
 					(unit 1)
 				)
@@
 		(on_board yes)
 		(dnp no)
-		(property "Reference" "#PWR0142"
+		(property "Reference" "#PWR0143"
 			(at 809.752 57.912 0)
 			(effects
@@
 			(project "ECU-techPorsche88"
 				(path "/2a08f213-b835-4bb3-95c3-61aa4df68063"
-					(reference "#PWR0142")
+					(reference "#PWR0143")
 					(unit 1)
 				)
@@
 		(on_board yes)
 		(dnp no)
-		(property "Reference" "#PWR0143"
+		(property "Reference" "#PWR0142"
 			(at 798.83 541.02 0)
 			(effects
@@
 			(project "ECU-techPorsche88"
 				(path "/2a08f213-b835-4bb3-95c3-61aa4df68063"
-					(reference "#PWR0143")
+					(reference "#PWR0142")
 					(unit 1)
 				)
@@
 		(on_board yes)
 		(dnp no)
-		(property "Reference" "#PWR042"
+		(property "Reference" "#PWR043"
 			(at 353.822 399.542 0)
 			(effects
@@
 			(project "ECU-techPorsche88"
 				(path "/2a08f213-b835-4bb3-95c3-61aa4df68063"
-					(reference "#PWR042")
+					(reference "#PWR043")
 					(unit 1)
 				)
